File: PCB/Project-24-7.kicad_sch (KiCad schematic)
At the start: 4 parts, among them U1 ESP32-C3, Y1 Crystal_40MHz

Commit message: Added LDO, Decoupling Caps & Antenna
Parts:
- added AE1: Antenna_Dipole, symbol Device:Antenna_Dipole
- added C10: 10n, symbol Device:C_Small
- added C11, C13, C6, C9: 1u, symbol Device:C_Small
- added C12, C5, C8: 100n, symbol Device:C_Small
- added C14, C15: 2p, symbol Device:C_Small
- added C3, C4, C7: 10u, symbol Device:C_Small
- added R1: 0R, symbol Device:R_Small
- added U2: ME6211C50M5, Package_TO_SOT_SMD:SOT-23-5, symbol Regulator_Linear:ME6211C50M5
- C1, C2: value 10p -> 15p
Connections:
- net GND: now also C10.2, C11.1, C12.2, C13.2, C14.2, C15.2, C3.2, C4.2, C5.1, C6.1, C7.1, C8.2, C9.2, U2.2 (V_{SS})
- net at U1.1 (LNA_IN): now also C14.1, R1.1
- net SCL: now reaches U1.10 (MTDI)
- net 3V3: now reaches U1.11 (VDD3P3_RTC)
- net 3V3: now also U1.17 (VDD3P3_CPU), U1.18 (VDD_SPI), U1.2 (VDD3P3), U1.3 (VDD3P3), U1.31 (VDDA), U1.32 (VDDA), C10.1, C11.2, C12.1, C13.1, C3.1, C5.2, C6.2, C7.2, C8.1, C9.1, U2.5 (V_{OUT})
- net SDA: now reaches U1.9 (MTMS)
- new net: AE1.1, C15.1, R1.2
- new net VBAT: C4.1, U2.1 (V_{IN}), U2.3 (CE)
